File: KiCad/sensor-de-movimiento/sensor-de-movimiento.kicad_pcb (KiCad board)
At the start: 2 copper layers, 50 x 50 mm, 3 parts, among them J1 Conector PIR, J2 Conector Bateria, U1 NodeMCU-32S

Commit message: Errores en KiCad
Parts:
- moved J2 16.8 mm to (131.6, 96.5)
- moved J1 11.3 mm to (137.7, 100.6), turned to 180 degrees
- moved U1 5.08 mm to (161.0, 97.5), turned to 0 degrees
Connections:
- U1 pad 14: Net-(U1-Pad14) -> GND
- U1 pad 19: Net-(U1-Pad19) -> +BATT
- U1 pad 32: Net-(U1-Pad32) -> GND
Routing:
- net Net-(J1-Pad2): track 89.0 -> 23.3 mm
- net GND: track 61.6 -> 88.4 mm
- net +BATT: track 27.4 -> 35.3 mm
